File: BackPCB/110ADR-BackPCB.kicad_pcb (KiCad board)
At the start: 2 copper layers, 440.3 x 124.8 mm, 0 parts

Commit message: cleanup and swapped MCU to PGA2040 on solder version as experiment.
Other:
- board text added: "110ADR-S"
- board text removed: "110ADR-HS"
