File: SwitchPlate/SwitchPlate.kicad_pcb (KiCad board)
At the start: 2 copper layers, 429.5 x 133.3 mm, 11 parts

Commit message: Modified Kicad Projects to make generating DXFs for laser cutting easier.
Parts:
- H1, H10, H2, H3, H4, H5, H6, H7, H8, H9: footprint MountingHole:MountingHole_2.2mm_M2 -> logo:MountingHole_2.2mm_M2_modified

Commit message: Made some tweaks to allow for easier Gerber generation
Routing:
- added copper zone on B.Cu, net (none)
- added copper zone on F.Cu, net (none)
- removed copper zone on B.Cu, net GND
- removed copper zone on F.Cu, net GND
Other:
- board size 429.5 x 133.3 mm -> 432.6 x 139.3 mm
