File: SwitchPlate/110ADR-SwitchPlate.kicad_pcb (KiCad board)
At the start: 2 copper layers, 429.5 x 125 mm, 14 parts

Commit message: padded switch plate and generated gerber for test price (£19.43)
Parts:
- removed G***: LOGO, logo:logo
Other:
- board size 429.5 x 125 mm -> 431.6 x 127.7 mm

Commit message: forgot to commit this change lol.
Parts:
- added G***: LOGO, logo:logo, F.Cu at (445.0, 63.0)

Commit message: Various fixes to clearances and fixed a lot of traces
Parts:
- removed H1, H10, H12, H13, H14, H2, H3, H4, H5, H6, H7, H8, H9: MountingHole, MountingHole:MountingHole_2.2mm_M2_Pad
Other:
- board size 431.6 x 127.7 mm -> 440.3 x 124.8 mm
- net class Default removed
