File: MainPCB/EnvKB110ADR.sch (KiCad schematic (older format))
At the start: 272 parts, among them J2 EVQPU, J5 Conn_01x03_Male, U1 TLV75533PDBVR, U3 RP2040, Y1 3225_4P

Commit message: Replaced flash with smaller uson-8 3x2 + regenerated Gerbers
Parts:
- FLASH1: value W25Q128JVPIQ -> W25Q16FWUXIE; footprint Package_SON:WSON-8-1EP_6x5mm_P1.27mm_EP3.4x4mm -> Package_SON:SON-8-1EP_3x2mm_P0.5mm_EP1.4x1.6mm
Changed lines of the file:
@@
 P 3100 5250
 F 0 "FLASH1" H 3100 5250 50  0000 C CNN
-F 1 "W25Q128JVPIQ" H 3100 4750 50  0000 C CNN
-F 2 "Package_SON:WSON-8-1EP_6x5mm_P1.27mm_EP3.4x4mm" H 3100 5250 50  0001 L BNN
+F 1 "W25Q16FWUXIE" H 3100 4750 50  0000 C CNN
+F 2 "Package_SON:SON-8-1EP_3x2mm_P0.5mm_EP1.4x1.6mm" H 3100 5250 50  0001 L BNN
 F 3 "" H 3100 5250 50  0001 L BNN
 F 4 "  " H 3100 5250 50  0001 C CNN "LCSC"
