File: MainPCB-STM32/EnvKB110ADR-STM32.kicad_pcb (KiCad board)
At the start: 2 copper layers, 429.5 x 125 mm, 249 parts, among them J1 Conn_01x03, SW1 Boot Mode, SW2 Reset Switch, U1 XC6206PxxxMR, U2 STM32F411CEUx, Y1 3225_4P 32.768khz

Commit message: Generated updated Gerber
Parts:
- added G***: LOGO, logo:lyra, F.Cu at (404.4, 65.8)
Other:
- board text added: "Envious.Design"
- board text removed: "Designed by"
