File: MainPCB-RPI+IOX/EnvKB105-RPI.kicad_pcb (KiCad board)
At the start: 2 copper layers, 429.5 x 125 mm, 251 parts, among them U1 Pico, U3 MCP23017_ML

Commit message: fixed ref and generated updated gerber
Parts:
- renumbered D_ANSI_1 to D_117
Changed lines of the file:
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@@
     (property "Sheetname" "")
     (attr smd)
-    (fp_text reference "D_ANSI_1" (at 0 2 90) (layer "B.SilkS")
+    (fp_text reference "D_117" (at 0 2 90) (layer "B.SilkS")
       (effects (font (size 1 1) (thickness 0.15)) (justify mirror))
     )
