File: MainPCB-RPI+IOX/EnvKB105-RPI.kicad_pcb (KiCad board)
At the start: 2 copper layers, 429.5 x 125 mm, 251 parts, among them U1 Pico, U3 MCP23017_ML

Commit message: sorted reference out
Routing:
- net unconnected-(U2-Pad16): vias 0 -> 1
- net GND: vias 1 -> 0
Changed lines of the file:
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@@
   (net 147 "unconnected-(USB1-PadA8)")
   (net 148 "unconnected-(USB1-PadB8)")
-  (net 149 "Net-(D_ANSI_1-Pad2)")
+  (net 149 "Net-(D_117-Pad2)")
   (net 150 "unconnected-(H1-Pad1)")
   (net 151 "unconnected-(H2-Pad1)")
@@
   (net 186 "unconnected-(U3-Pad2)")
   (net 187 "unconnected-(U3-Pad3)")
+  (net 188 "unconnected-(U2-Pad16)")
   (footprint "MountingHole:MountingHole_2.2mm_M2_Pad" (layer "F.Cu")
     (at 42.9 73.3)
@@
       (net 15 "col14") (pinfunction "COL") (pintype "passive"))
     (pad "2" thru_hole circle (at 2.54 -5.08 270) (size 3.25 3.25) (drill 3) (layers *.Cu *.Mask)
-      (net 149 "Net-(D_ANSI_1-Pad2)") (pinfunction "ROW") (pintype "passive"))
+      (net 149 "Net-(D_117-Pad2)") (pinfunction "ROW") (pintype "passive"))
     (pad "2" smd rect (at 4.34 -5.08 270) (size 5.5 2.5) (layers "B.Cu")
-      (net 149 "Net-(D_ANSI_1-Pad2)") (pinfunction "ROW") (pintype "passive"))
+      (net 149 "Net-(D_117-Pad2)") (pinfunction "ROW") (pintype "passive"))
   )
   (footprint "EnvExtras:MXOnly-1U-Hotswap-Modified" (layer "F.Cu")
@@
       (net 25 "row4") (pinfunction "K") (pintype "passive"))
     (pad "2" smd rect (at 1.65 0 270) (size 0.9 1.2) (layers "B.Cu" "B.Paste" "B.Mask")
-      (net 149 "Net-(D_ANSI_1-Pad2)") (pinfunction "A") (pintype "passive"))
+      (net 149 "Net-(D_117-Pad2)") (pinfunction "A") (pintype "passive"))
     (model "${KICAD6_3DMODEL_DIR}/Diode_SMD.3dshapes/D_SOD-123.wrl"
       (offset (xyz 0 0 0))
@@
   (segment (start 443.63 168.76) (end 444.4 167.99) (width 0.15) (layer "B.Cu") (net 133))
   (segment (start 444.4 167.99) (end 444.4 161.678) (width 0.15) (layer "B.Cu") (net 133))
-  (via (at 393.25 71) (size 0.8) (drill 0.4) (layers "F.Cu" "B.Cu") (net 135))
   (segment (start 404.0875 76.6) (end 403.2 76.6) (width 0.25) (layer "B.Cu") (net 135))
   (segment (start 402.55 73.35) (end 401.25 74.65) (width 0.25) (layer "B.Cu") (net 135))
@@
   (segment (start 300.7 109.55) (end 300.7 110.2) (width 0.15) (layer "B.Cu") (net 149))
   (segment (start 312.38 114.8) (end 314.14 113.04) (width 0.15) (layer "B.Cu") (net 149))
+  (via (at 393.25 71) (size 0.8) (drill 0.4) (layers "F.Cu" "B.Cu") (net 188))
   (zone (net 135) (net_name "GND") (layers F&B.Cu) (hatch edge 0.508)
     (connect_pads yes (clearance 0.127))

Commit message: swapped IO expander package to DIP
Parts:
- removed U3: MCP23017_ML, Package_DFN_QFN:QFN-28-1EP_6x6mm_P0.65mm_EP4.25x4.25mm
- added C1: 0.1uf, Capacitor_SMD:C_0805_2012Metric, B.Cu at (390.1, 63.4)
- added R1: 330r, Resistor_SMD:R_0805_2012Metric, B.Cu at (390.1, 61.3)
- added U2: MCP23017_SP, Package_DIP:DIP-28_W7.62mm, B.Cu at (369.6, 69.4)
- moved H9 308.4 mm to (138.6, 32.9)
- moved H5 238.2 mm to (209.1, 98.7)
- moved kibuzzard-6261CED5 10.6 mm to (138.9, 164.4)
Connections:
- U1 pad 21: row1 -> unconnected-(U1-Pad21)
- USB1 pad S1: GND -> Net-(USB1-PadS1)
Routing:
- net col5: track 363.6 -> 334.1 mm
- net Net-(USB1-PadS1): track 0.00 -> 28.1 mm
- net col0: track 509.9 -> 482.9 mm
- net col6: track 336.8 -> 310.0 mm
- net col1: track 424.5 -> 400.2 mm
- net col7: track 328.9 -> 305.0 mm
- net col2: track 421.6 -> 399.5 mm
- net col8: track 310.7 -> 289.2 mm
- net row1: track 355.6 -> 334.2 mm, vias 1 -> 0
- net col9: track 292.1 -> 271.4 mm
- net col3: track 426.1 -> 406.8 mm
- net col10: track 294.6 -> 275.5 mm
- net col11: track 272.3 -> 255.0 mm
- net VBUS: track 29.9 -> 13.1 mm, vias 3 -> 2
- net VSYS: track 62.0 -> 78.8 mm, vias 0 -> 1
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Other:
- board text added: "Oh Henlo there...."

Commit message: Added position for OLED and RGB indicator LEDs among other things
Parts:
- added J1: Conn_01x04, Connector_PinHeader_2.54mm:PinHeader_1x04_P2.54mm_Vertical, F.Cu at (462.9, 63.4)
- added rgb1: SK6812MINI, LED_SMD:LED_SK6812MINI_PLCC4_3.5x3.5mm_P1.75mm, F.Cu at (414.3, 62.3)
- added rgb2: SK6812MINI, LED_SMD:LED_SK6812MINI_PLCC4_3.5x3.5mm_P1.75mm, F.Cu at (421.9, 62.3)
- added rgb3: SK6812MINI, LED_SMD:LED_SK6812MINI_PLCC4_3.5x3.5mm_P1.75mm, F.Cu at (414.3, 67.3)
- added rgb4: SK6812MINI, LED_SMD:LED_SK6812MINI_PLCC4_3.5x3.5mm_P1.75mm, F.Cu at (421.9, 67.3)
- added rgb5: SK6812MINI, LED_SMD:LED_SK6812MINI_PLCC4_3.5x3.5mm_P1.75mm, F.Cu at (414.3, 72.3)
- added rgb6: SK6812MINI, LED_SMD:LED_SK6812MINI_PLCC4_3.5x3.5mm_P1.75mm, F.Cu at (421.9, 72.3)
- moved H9 70.3 mm to (113.8, 98.7)
- moved G*** 67.8 mm to (374.8, 126.2)
Connections:
- U1 pad 34: unconnected-(U1-Pad34) -> GP28-LED
Routing:
- net VSYS: track 78.8 -> 177.2 mm
- net GP28-LED: track 0.00 -> 30.8 mm
- net I2C_SCL-1: track 61.5 -> 79.6 mm
- net Net-(rgb4-Pad1): track 0.00 -> 14.3 mm
- net Net-(rgb2-Pad1): track 0.00 -> 14.3 mm
- net I2C_SDA-1: track 61.4 -> 67.2 mm
- net col4: track 366.4 -> 371.4 mm
- net Net-(rgb5-Pad1): track 0.00 -> 4.41 mm
- net Net-(rgb3-Pad1): track 0.00 -> 4.41 mm
- net Net-(rgb1-Pad1): track 0.00 -> 4.41 mm
- net USB_D+: track 102.0 -> 102.8 mm, vias 2 -> 0
Other:
- outline, holes or cut-outs redrawn
- board text added: "ADC0"
- board text added: "ADC1"
- board text added: "CSn"
- board text added: "GND"
- board text added: "GND VSYS SCL SDA"
- board text added: "General"
- board text added: "I2C"
- board text added: "RUN"
- board text added: "RX"
- board text added: "SCK"
- board text added: "SCL"
- board text added: "SDA"
- board text added: "SPI"
- board text added: "Spare GPIOs"
- board text added: "TX"
- board text added: "UART"
- board text removed: "BlackCatPlasticWorks.com"
