File: MainPCB-RPI+IOX/EnvKB105-RPI.kicad_pcb (KiCad board)
At the start: 2 copper layers, 429.5 x 125 mm, 260 parts, among them J1 Conn_01x04, U1 Pico, U2 MCP23017_SP

Commit message: some adjustments to make CAD a bit easier
Parts:
- H1, H10, H11, H12, H13, H14, H15, H16, H17, H18, H2, H3, H4, H5, H6, H7, H8, H9: footprint MountingHole:MountingHole_2.2mm_M2_Pad -> EnvExtras:MountingHole_2.2mm_M2_Pad-Mod

Commit message: Changed my mind on Mount holes
Parts:
- removed H10, H11, H12, H13, H14, H15, H16, H17, H18: MountingHole, EnvExtras:MountingHole_2.2mm_M2_Pad-Mod
- moved H4 377.8 mm to (90.0, 119.0)
- moved H3 377.8 mm to (403.3, 69.9)
- moved H9 319.5 mm to (428.1, 155.7)
- moved H2 210.8 mm to (252.3, 72.4)
- moved H8 179.7 mm to (253.0, 156.3)
- moved H7 111.2 mm to (86.7, 157.4)
- moved H6 111.0 mm to (409.1, 118.2)
- moved H1 48.7 mm to (91.6, 72.4)
- moved H5 47.6 mm to (252.5, 118.2)
- moved U2 4.12 mm to (365.5, 69.4)
- moved D_108 3.53 mm to (248.8, 164.5)
Connections:
- H1 pad 1: unconnected-(H1-Pad1) -> (no net)
- H2 pad 1: unconnected-(H2-Pad1) -> (no net)
- H3 pad 1: unconnected-(H3-Pad1) -> (no net)
- H4 pad 1: unconnected-(H4-Pad1) -> (no net)
- H5 pad 1: unconnected-(H5-Pad1) -> (no net)
- H6 pad 1: unconnected-(H6-Pad1) -> (no net)
- H7 pad 1: unconnected-(H7-Pad1) -> (no net)
- H8 pad 1: unconnected-(H8-Pad1) -> (no net)
- H9 pad 1: unconnected-(H9-Pad1) -> (no net)
Routing:
- net I2C_SCL-1: track 79.6 -> 85.5 mm
- net I2C_SDA-1: track 67.2 -> 72.9 mm
- net col8: track 289.2 -> 284.3 mm
- net col1: track 400.2 -> 396.1 mm
- net col5: track 334.1 -> 329.9 mm
- net col9: track 271.4 -> 267.3 mm
- net col7: track 305.0 -> 300.9 mm
- net col6: track 310.0 -> 305.8 mm
- net col4: track 371.4 -> 367.3 mm
- net col2: track 399.5 -> 395.3 mm
- net col12: track 195.5 -> 191.4 mm
- net VSYS: track 177.2 -> 181.3 mm
- net col3: track 406.8 -> 402.6 mm
- net col0: track 482.9 -> 479.1 mm
- net row4: track 476.2 -> 479.9 mm
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Other:
- board text added: "Oh Henlo there.... I am a MCP23017!"
- board text removed: "Oh Henlo there...."

Commit message: added 7u bottom and stepped capslock
Parts:
- added K_104B1: KEYSW, EnvExtras:MXOnly-1U-Hotswap-Modified, F.Cu at (51.9, 165.8)
- added K_105B1: KEYSW, EnvExtras:MXOnly-1U-Hotswap-Modified, F.Cu at (75.7, 165.8)
- added K_106B1: KEYSW, EnvExtras:MXOnly-1U-Hotswap-Modified, F.Cu at (99.5, 165.8)
- added K_107B1: KEYSW, EnvExtras:MXOnly-1U-Hotswap-Modified, F.Cu at (180.4, 165.8)
- added K_108B1: KEYSW, EnvExtras:MXOnly-1U-Hotswap-Modified, F.Cu at (260.6, 165.8)
- added K_109B1: KEYSW, EnvExtras:MXOnly-1U-Hotswap-Modified, F.Cu at (282.9, 165.8)
- added K_111B1: KEYSW, EnvExtras:MXOnly-1U-Hotswap-Modified, F.Cu at (309.0, 165.8)
- added K_70B1: KEYSW, EnvExtras:MXOnly-1U-Hotswap-Modified, F.Cu at (49.5, 127.7)
- added stab101: MountingHole, Mounting_Keyboard_Stabilizer:Stabilizer_Cherry_MX_7u, F.Cu at (180.4, 165.8)
- moved D_107 14.0 mm to (191.1, 167.3)
- moved D_106 6.46 mm to (110.2, 161.2)
- moved D_104 6.22 mm to (61.4, 161.2), turned to 180 degrees
- moved D_105 3.95 mm to (85.6, 163.7)
- moved D_109 1.90 mm to (274.6, 165.4)
- moved D_110 1.25 mm to (298.5, 166.1)
Routing:
- net row7: track 514.7 -> 579.0 mm
- net col0: track 479.1 -> 508.2 mm
- net Net-(D_70-Pad2): track 11.7 -> 37.0 mm
- net Net-(D_105-Pad2): track 6.78 -> 31.8 mm
- net Net-(D_107-Pad2): track 5.96 -> 30.7 mm
- net Net-(D_106-Pad2): track 6.66 -> 31.1 mm
- net Net-(D_104-Pad2): track 6.97 -> 30.7 mm
- net Net-(D_109-Pad2): track 6.97 -> 30.6 mm
- net col6: track 305.8 -> 329.5 mm
- net Net-(D_110-Pad2): track 6.97 -> 30.6 mm
- net Net-(D_111-Pad2): track 6.97 -> 26.7 mm
- net col1: track 396.1 -> 412.5 mm
- net col3: track 402.6 -> 418.8 mm
- net col13: track 243.1 -> 257.9 mm
- net col11: track 254.9 -> 267.5 mm
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Other:
- board text added: "Upside down switch positions on this row are for 7u spacebar."
- board text removed: "Kailh makes pink hotswap sockets and I'm upset I don't have any."
