File: MainPCB-RPI+IOX/EnvKB105-RPI.kicad_sch (KiCad schematic)
At the start: 256 parts, among them J1 Conn_01x04, U1 Pico, U2 MCP23017_SP

Commit message: some general tweaks and preparation for ordering
Parts:
- added H12, H4, H8: MountingHole, EnvExtras:MountingHole_2.2mm_M2_Pad-Mod, symbol Mechanical:MountingHole
- renumbered H8 to H10, H9 to H11, H4 to H5, H5 to H6, H6 to H7, H7 to H9
Changed lines of the file:
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@@
+    )
+  )
+  (symbol (lib_id "Mechanical:MountingHole") (at 57.785 205.105 0) (unit 1)
+    (in_bom yes) (on_board yes)
+    (property "Reference" "H12" (id 0) (at 56.515 201.93 0)
+      (effects (font (size 1.27 1.27)) (justify left))
+    )
+    (property "Value" "MountingHole" (id 1) (at 60.96 206.3749 0)
+      (effects (font (size 1.27 1.27)) (justify left) hide)
+    )
+    (property "Footprint" "EnvExtras:MountingHole_2.2mm_M2_Pad-Mod" (id 2) (at 57.785 205.105 0)
+      (effects (font (size 1.27 1.27)) hide)
+    )
+    (property "Datasheet" "~" (id 3) (at 57.785 205.105 0)
+      (effects (font (size 1.27 1.27)) hide)
     )
   )
@@
   (symbol (lib_id "Mechanical:MountingHole") (at 47.625 199.39 0) (unit 1)
     (in_bom yes) (on_board yes)
-    (property "Reference" "H5" (id 0) (at 46.355 196.215 0)
+    (property "Reference" "H6" (id 0) (at 46.355 196.215 0)
       (effects (font (size 1.27 1.27)) (justify left))
     )
@@
     )
     (property "Datasheet" "~" (id 3) (at 47.625 199.39 0)
+      (effects (font (size 1.27 1.27)) hide)
+    )
+  )
+  (symbol (lib_id "Mechanical:MountingHole") (at 57.785 193.675 0) (unit 1)
+    (in_bom yes) (on_board yes)
+    (property "Reference" "H4" (id 0) (at 56.515 190.5 0)
+      (effects (font (size 1.27 1.27)) (justify left))
+    )
+    (property "Value" "MountingHole" (id 1) (at 60.96 194.9449 0)
+      (effects (font (size 1.27 1.27)) (justify left) hide)
+    )
+    (property "Footprint" "EnvExtras:MountingHole_2.2mm_M2_Pad-Mod" (id 2) (at 57.785 193.675 0)
+      (effects (font (size 1.27 1.27)) hide)
+    )
+    (property "Datasheet" "~" (id 3) (at 57.785 193.675 0)
       (effects (font (size 1.27 1.27)) hide)
     )
@@
   (symbol (lib_id "Mechanical:MountingHole") (at 42.545 199.39 0) (unit 1)
     (in_bom yes) (on_board yes)
-    (property "Reference" "H4" (id 0) (at 41.275 196.215 0)
+    (property "Reference" "H5" (id 0) (at 41.275 196.215 0)
       (effects (font (size 1.27 1.27)) (justify left))
     )
@@
     (pin "2")
   )
+  (symbol (lib_id "Mechanical:MountingHole") (at 57.785 199.39 0) (unit 1)
+    (in_bom yes) (on_board yes)
+    (property "Reference" "H8" (id 0) (at 56.515 196.215 0)
+      (effects (font (size 1.27 1.27)) (justify left))
+    )
+    (property "Value" "MountingHole" (id 1) (at 60.96 200.6599 0)
+      (effects (font (size 1.27 1.27)) (justify left) hide)
+    )
+    (property "Footprint" "EnvExtras:MountingHole_2.2mm_M2_Pad-Mod" (id 2) (at 57.785 199.39 0)
+      (effects (font (size 1.27 1.27)) hide)
+    )
+    (property "Datasheet" "~" (id 3) (at 57.785 199.39 0)
+      (effects (font (size 1.27 1.27)) hide)
+    )
+  )
   (symbol (lib_id "MX_Alps_Hybrid:MX-NoLED") (at 49.53 524.51 0) (unit 1)
     (in_bom yes) (on_board yes)
@@
   (symbol (lib_id "Mechanical:MountingHole") (at 52.705 205.105 0) (unit 1)
     (in_bom yes) (on_board yes)
-    (property "Reference" "H9" (id 0) (at 51.435 201.93 0)
+    (property "Reference" "H11" (id 0) (at 51.435 201.93 0)
       (effects (font (size 1.27 1.27)) (justify left))
     )
@@
   (symbol (lib_id "Mechanical:MountingHole") (at 47.625 205.105 0) (unit 1)
     (in_bom yes) (on_board yes)
-    (property "Reference" "H8" (id 0) (at 46.355 201.93 0)
+    (property "Reference" "H10" (id 0) (at 46.355 201.93 0)
       (effects (font (size 1.27 1.27)) (justify left))
     )
@@
   (symbol (lib_id "Mechanical:MountingHole") (at 52.705 199.39 0) (unit 1)
     (in_bom yes) (on_board yes)
-    (property "Reference" "H6" (id 0) (at 51.435 196.215 0)
+    (property "Reference" "H7" (id 0) (at 51.435 196.215 0)
       (effects (font (size 1.27 1.27)) (justify left))
     )
@@
   (symbol (lib_id "Mechanical:MountingHole") (at 42.545 205.105 0) (unit 1)
     (in_bom yes) (on_board yes)
-    (property "Reference" "H7" (id 0) (at 41.275 201.93 0)
+    (property "Reference" "H9" (id 0) (at 41.275 201.93 0)
       (effects (font (size 1.27 1.27)) (justify left))
     )
@@
       (reference "H3") (unit 1) (value "MountingHole") (footprint "EnvExtras:MountingHole_2.2mm_M2_Pad-Mod")
     )
+    (path "/63973fad-1b00-4427-8128-c3ce1c8dc02d"
+      (reference "H4") (unit 1) (value "MountingHole") (footprint "EnvExtras:MountingHole_2.2mm_M2_Pad-Mod")
+    )
     (path "/7fff0109-adb9-48ca-ba9c-e1fca4eeff5f"
-      (reference "H4") (unit 1) (value "MountingHole") (footprint "EnvExtras:MountingHole_2.2mm_M2_Pad-Mod")
+      (reference "H5") (unit 1) (value "MountingHole") (footprint "EnvExtras:MountingHole_2.2mm_M2_Pad-Mod")
     )
     (path "/627ae846-a75d-47d6-8420-934904a05713"
-      (reference "H5") (unit 1) (value "MountingHole") (footprint "EnvExtras:MountingHole_2.2mm_M2_Pad-Mod")
+      (reference "H6") (unit 1) (value "MountingHole") (footprint "EnvExtras:MountingHole_2.2mm_M2_Pad-Mod")
     )
     (path "/d199f85a-e3d2-475e-9d74-e800d7f88d5b"
-      (reference "H6") (unit 1) (value "MountingHole") (footprint "EnvExtras:MountingHole_2.2mm_M2_Pad-Mod")
+      (reference "H7") (unit 1) (value "MountingHole") (footprint "EnvExtras:MountingHole_2.2mm_M2_Pad-Mod")
+    )
+    (path "/a6e68e3e-7142-46bc-8c0f-69cde6683553"
+      (reference "H8") (unit 1) (value "MountingHole") (footprint "EnvExtras:MountingHole_2.2mm_M2_Pad-Mod")
     )
     (path "/d57b711d-5551-4b72-bb9b-62a4bf3eee54"
-      (reference "H7") (unit 1) (value "MountingHole") (footprint "EnvExtras:MountingHole_2.2mm_M2_Pad-Mod")
+      (reference "H9") (unit 1) (value "MountingHole") (footprint "EnvExtras:MountingHole_2.2mm_M2_Pad-Mod")
     )
     (path "/b513d15e-d1e8-4baa-8757-c1baec808360"
-      (reference "H8") (unit 1) (value "MountingHole") (footprint "EnvExtras:MountingHole_2.2mm_M2_Pad-Mod")
+      (reference "H10") (unit 1) (value "MountingHole") (footprint "EnvExtras:MountingHole_2.2mm_M2_Pad-Mod")
     )
     (path "/b3d37140-363f-4760-8027-80c36ea35ba0"
-      (reference "H9") (unit 1) (value "MountingHole") (footprint "EnvExtras:MountingHole_2.2mm_M2_Pad-Mod")
+      (reference "H11") (unit 1) (value "MountingHole") (footprint "EnvExtras:MountingHole_2.2mm_M2_Pad-Mod")
+    )
+    (path "/01c9ca24-50d0-4739-97a0-7d6aae335f31"
+      (reference "H12") (unit 1) (value "MountingHole") (footprint "EnvExtras:MountingHole_2.2mm_M2_Pad-Mod")
     )
     (path "/3305d520-5042-4ed2-bc41-b5590d18bb4d"
