File: MainPCB-RP2040/EnvKB110ADR-RP2040.kicad_pcb (KiCad board)
At the start: 2 copper layers, 429.5 x 125 mm, 290 parts, among them J2 EVQPU, J5 Conn_01x03_Male, U1 TLV75533PDBVR, U3 RP2040, Y1 3225_4P

Commit message: generated updated gerber
Parts:
- moved D_ANSI_1 1.10 mm to (300.7, 107.9)
Routing:
- net Net-(D_ANSI_1-Pad2): track 20.1 -> 21.3 mm
Changed lines of the file:
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@@
     (pad "2" smd rect locked (at -2.625 -0.85) (size 1.55 1) (layers "B.Cu" "B.Paste" "B.Mask")
       (net 135 "GND") (pinfunction "2") (pintype "passive"))
-    (model "${KISYS3DMOD}/Button_Switch_SMD.3dshapes/Panasonic_EVQPUJ_EVQPUA.wrl"
+    (model "C:/Users/Envy/Documents/GitHub/_RESOURCES/EVQ-P7J01P--3DModel-STEP-56544.STEP"
       (offset (xyz 0 0 0))
       (scale (xyz 1 1 1))
-      (rotate (xyz 0 0 0))
+      (rotate (xyz -90 0 180))
     )
   )
@@
     (pad "2" smd rect locked (at 2.625 -0.85) (size 1.55 1) (layers "B.Cu" "B.Paste" "B.Mask")
       (net 160 "/RUN") (pinfunction "2") (pintype "passive"))
-    (model "${KISYS3DMOD}/Button_Switch_SMD.3dshapes/Panasonic_EVQPUJ_EVQPUA.wrl"
+    (model "C:/Users/Envy/Documents/GitHub/_RESOURCES/EVQ-P7J01P--3DModel-STEP-56544.STEP"
       (offset (xyz 0 0 0))
       (scale (xyz 1 1 1))
-      (rotate (xyz 0 0 0))
+      (rotate (xyz -90 0 180))
     )
   )
@@
   )
   (footprint "Diode_SMD:D_SOD-123" (layer "B.Cu")
-    (at 300.7 109 -90)
+    (at 300.7 107.9 -90)
     (descr "SOD-123")
     (tags "SOD-123")
@@
   (via (at 406.40292 111.844526) (size 0.8) (drill 0.4) (layers "F.Cu" "B.Cu") (net 25))
   (segment (start 445.83 114.68) (end 443 111.85) (width 0.15) (layer "B.Cu") (net 25))
-  (segment (start 321.9 102) (end 315.7 102) (width 0.15) (layer "B.Cu") (net 25))
-  (segment (start 324.8 104.9) (end 321.9 102) (width 0.15) (layer "B.Cu") (net 25))
+  (segment (start 346.1625 111.85) (end 327.75 111.85) (width 0.15) (layer "B.Cu") (net 25))
   (segment (start 315.7 102) (end 312.3 98.6) (width 0.15) (layer "B.Cu") (net 25))
-  (segment (start 327.75 111.85) (end 324.8 108.9) (width 0.15) (layer "B.Cu") (net 25))
-  (segment (start 300.7 103.5) (end 300.7 107.35) (width 0.15) (layer "B.Cu") (net 25))
+  (segment (start 296.2 111.85) (end 300.7 107.35) (width 0.15) (layer "B.Cu") (net 25))
+  (segment (start 300.7 107.35) (end 300.7 106.25) (width 0.15) (layer "B.Cu") (net 25))
   (segment (start 419.229078 64.21802) (end 419.661058 64.65) (width 0.15) (layer "B.Cu") (net 25))
   (segment (start 407.61 72.16) (end 407.61 70.472398) (width 0.15) (layer "B.Cu") (net 25))
+  (segment (start 324.8 108.9) (end 324.8 104.9) (width 0.15) (layer "B.Cu") (net 25))
+  (segment (start 312.3 98.6) (end 305.6 98.6) (width 0.15) (layer "B.Cu") (net 25))
   (segment (start 407.61 70.472398) (end 413.864378 64.21802) (width 0.15) (layer "B.Cu") (net 25))
+  (segment (start 327.75 111.85) (end 324.8 108.9) (width 0.15) (layer "B.Cu") (net 25))
+  (segment (start 321.9 102) (end 315.7 102) (width 0.15) (layer "B.Cu") (net 25))
+  (segment (start 293.775 111.85) (end 296.2 111.85) (width 0.15) (layer "B.Cu") (net 25))
   (segment (start 445.8 114.71) (end 445.83 114.68) (width 0.15) (layer "B.Cu") (net 25))
   (segment (start 293.775 111.85) (end 65.175 111.85) (width 0.15) (layer "B.Cu") (net 25))
+  (segment (start 300.7 103.5) (end 300.7 106.25) (width 0.15) (layer "B.Cu") (net 25))
   (segment (start 413.864378 64.21802) (end 419.229078 64.21802) (width 0.15) (layer "B.Cu") (net 25))
   (segment (start 419.661058 64.65) (end 423.3625 64.65) (width 0.15) (layer "B.Cu") (net 25))
   (segment (start 445.8 118.76) (end 445.8 114.71) (width 0.15) (layer "B.Cu") (net 25))
-  (segment (start 296.2 111.85) (end 300.7 107.35) (width 0.15) (layer "B.Cu") (net 25))
-  (segment (start 305.6 98.6) (end 300.7 103.5) (width 0.15) (layer "B.Cu") (net 25))
-  (segment (start 312.3 98.6) (end 305.6 98.6) (width 0.15) (layer "B.Cu") (net 25))
   (segment (start 443 111.85) (end 346.1625 111.85) (width 0.15) (layer "B.Cu") (net 25))
   (segment (start 450.77 123.73) (end 445.8 118.76) (width 0.15) (layer "B.Cu") (net 25))
-  (segment (start 346.1625 111.85) (end 327.75 111.85) (width 0.15) (layer "B.Cu") (net 25))
-  (segment (start 324.8 108.9) (end 324.8 104.9) (width 0.15) (layer "B.Cu") (net 25))
-  (segment (start 293.775 111.85) (end 296.2 111.85) (width 0.15) (layer "B.Cu") (net 25))
+  (segment (start 305.6 98.6) (end 300.7 103.5) (width 0.15) (layer "B.Cu") (net 25))
+  (segment (start 324.8 104.9) (end 321.9 102) (width 0.15) (layer "B.Cu") (net 25))
   (segment (start 406.016841 132.951921) (end 406.016841 130.655759) (width 0.15) (layer "F.Cu") (net 26))
   (segment (start 407.26144 129.41116) (end 407.26144 111.622416) (width 0.15) (layer "F.Cu") (net 26))
@@
   (segment (start 443.63 168.76) (end 444.4 167.99) (width 0.15) (layer "B.Cu") (net 133))
   (segment (start 444.4 167.99) (end 444.4 161.678) (width 0.15) (layer "B.Cu") (net 133))
-  (segment (start 431.675 63.45) (end 432.91 62.215) (width 0.15) (layer "F.Cu") (net 134))
+  (segment (start 431.675 63.45) (end 432.91 57.87) (width 0.15) (layer "F.Cu") (net 134))
   (segment (start 409.69 61.6) (end 419.38 61.6) (width 0.4) (layer "F.Cu") (net 134))
   (segment (start 420.25 62.47) (end 422.155 62.47) (width 0.35) (layer "F.Cu") (net 134))
   (segment (start 419.38 61.6) (end 420.25 62.47) (width 0.4) (layer "F.Cu") (net 134))
   (segment (start 422.155 62.47) (end 422.205 62.52) (width 0.35) (layer "F.Cu") (net 134))
-  (segment (start 432.91 62.215) (end 432.91 57.87) (width 0.15) (layer "F.Cu") (net 134))
   (via (at 422.205 62.52) (size 0.4) (drill 0.2) (layers "F.Cu" "B.Cu") (net 134))
   (via (at 420.25 62.47) (size 0.8) (drill 0.4) (layers "F.Cu" "B.Cu") (net 134))
@@
   (segment (start 431.218302 63.97502) (end 431.093282 63.85) (width 0.127) (layer "B.Cu") (net 161))
   (segment (start 310.8 114.8) (end 312.38 114.8) (width 0.15) (layer "B.Cu") (net 164))
+  (segment (start 300.7 110.2) (end 303.5 113) (width 0.15) (layer "B.Cu") (net 164))
   (segment (start 303.5 116.5) (end 304.9 117.9) (width 0.15) (layer "B.Cu") (net 164))
   (segment (start 304.9 117.9) (end 307.7 117.9) (width 0.15) (layer "B.Cu") (net 164))
-  (segment (start 312.38 114.8) (end 314.14 113.04) (width 0.15) (layer "B.Cu") (net 164))
-  (segment (start 301.15 110.65) (end 303.5 113) (width 0.15) (layer "B.Cu") (net 164))
   (segment (start 307.7 117.9) (end 310.8 114.8) (width 0.15) (layer "B.Cu") (net 164))
   (segment (start 303.5 113) (end 303.5 116.5) (width 0.15) (layer "B.Cu") (net 164))
+  (segment (start 300.7 109.55) (end 300.7 110.2) (width 0.15) (layer "B.Cu") (net 164))
+  (segment (start 312.38 114.8) (end 314.14 113.04) (width 0.15) (layer "B.Cu") (net 164))
   (segment (start 443.51 69.8525) (end 443.51 69) (width 0.127) (layer "F.Cu") (net 178))
   (segment (start 443 70.3625) (end 443.51 69.8525) (width 0.127) (layer "F.Cu") (net 178))

Commit message: various small adjustments
Parts:
- removed the G*** at (406.4, 66.2)
- removed the G*** at (368.9, 126.5)
- removed H10, H11, H12, H13, H14, H16, H17, H18, H3: MountingHole, MountingHole:MountingHole_2.2mm_M2_Pad
- added H5: MountingHole, MountingHole:MountingHole_2.2mm_M2_Pad, F.Cu at (252.5, 118.2)
- added H9: MountingHole, MountingHole:MountingHole_2.2mm_M2_Pad, F.Cu at (428.1, 155.7)
- moved H4 377.8 mm to (90.0, 119.0)
- moved H2 210.8 mm to (252.3, 72.4)
- moved H8 179.7 mm to (253.0, 156.3)
- moved H15 174.2 mm to (403.3, 69.9)
- moved H7 111.2 mm to (86.7, 157.4)
- moved H6 111.0 mm to (409.1, 118.2)
- moved H1 48.7 mm to (91.6, 72.4)
- moved J5 9.03 mm to (459.2, 55.6)
- moved D_69 6.31 mm to (458.7, 123.6)
- moved D_49 5.28 mm to (63.9, 105.1)
Routing:
- net row4: track 469.0 -> 484.8 mm
- net /SWD: track 31.6 -> 40.6 mm
- net /SWCLK: track 35.7 -> 44.7 mm
- net Net-(D_69-Pad2): track 14.6 -> 9.34 mm
- net row5: track 463.2 -> 467.6 mm
- net Net-(D_49-Pad2): track 9.49 -> 6.09 mm
- net col0: track 534.2 -> 536.8 mm
- net col11: track 312.8 -> 315.3 mm
- net col1: track 451.4 -> 453.7 mm
- net row7: track 504.2 -> 506.3 mm
- net row6: track 493.7 -> 495.6 mm
- net col2: track 448.6 -> 449.2 mm
- net VBUS: track 118.7 -> 118.2 mm
- net +3V3: vias 5 -> 4
