File: MainPCB - Solder Ver/EnvKB105-RPI.kicad_sch (KiCad schematic)
At the start: 285 parts, among them J2 Button, J5 Conn_01x03_Male, U1 SOT-23-5 5.5V 3.3V 500mA, U3 RP2040, Y1 3225_4P 12MHz

Commit message: generated Gerbers for solder version
Parts:
- renumbered RSW1 to BTTN1, J2 to BTTN2
Changed lines of the file:
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@@
   (symbol (lib_id "Switch:SW_Push") (at 144.78 165.1 0) (unit 1)
     (in_bom yes) (on_board yes) (dnp no)
-    (property "Reference" "RSW1" (at 144.78 170.18 0)
+    (property "Reference" "BTTN1" (at 144.78 170.18 0)
       (effects (font (size 1.27 1.27)))
     )
@@
       (project "EnvKB105-RPI"
         (path "/597a11f2-5d2c-4a65-ac95-38ad106e1367"
-          (reference "RSW1") (unit 1)
+          (reference "BTTN1") (unit 1)
         )
       )
@@
   (symbol (lib_id "Switch:SW_Push") (at 33.02 111.76 0) (mirror y) (unit 1)
     (in_bom yes) (on_board yes) (dnp no)
-    (property "Reference" "J2" (at 31.75 107.95 0)
+    (property "Reference" "BTTN2" (at 31.75 107.95 0)
       (effects (font (size 1.27 1.27)))
     )
@@
       (project "EnvKB105-RPI"
         (path "/597a11f2-5d2c-4a65-ac95-38ad106e1367"
-          (reference "J2") (unit 1)
-        )
-      )
+          (reference "BTTN2") (unit 1)
+        )
+      )

Commit message: cleanup and swapped MCU to PGA2040 on solder version as experiment.
Parts:
- removed BTTN1: TSA343G00-250J2, Button_Switch_SMD:SW_Push_SPST_NO_Alps_SKRK, symbol Switch:SW_Push
- removed BTTN2: Button, Button_Switch_SMD:SW_Push_SPST_NO_Alps_SKRK, symbol Switch:SW_Push
- removed C1, C17, C4, CBP1: 10uf 0402, Capacitor_SMD:C_0402_1005Metric, symbol Device:C
- removed C10, C102: 2.2uF 0402, Capacitor_SMD:C_0402_1005Metric, symbol Device:C
- removed C11, C13, C14, C15, C16, C18, C5, C6, C7, C8: 100nf 0402, Capacitor_SMD:C_0402_1005Metric, symbol Device:C
- removed C19, C2: 22pf 0402, Capacitor_SMD:C_0402_1005Metric, symbol Device:C
- removed C3: 1uf 0402, Capacitor_SMD:C_0402_1005Metric, symbol Device:C
- removed D1: 1N4002W, Diode_SMD:D_SOD-123, symbol Device:D_Schottky
- removed F1: 0805L050WR, Fuse:Fuse_0805_2012Metric, symbol Device:Polyfuse_Small
- removed FB1: FerriteBead 0402, Resistor_SMD:R_0402_1005Metric, symbol Device:FerriteBead_Small
- removed FLASH1: W25Q16JVUXIQ, Package_SON:SON-8-1EP_3x2mm_P0.5mm_EP1.4x1.6mm, symbol Memory_Flash:W25Q32JVZP
- removed R1, R11: 1K 0402, Resistor_SMD:R_0402_1005Metric, symbol Device:R
- removed R2: 10K 0402, Resistor_SMD:R_0402_1005Metric, symbol Device:R
- removed R3, R4: 27r 0402 resistor, Resistor_SMD:R_0402_1005Metric, symbol Device:R
- removed R7: 100K 0402, Resistor_SMD:R_0402_1005Metric, symbol Device:R
- removed U1: SOT-23-5 5.5V 3.3V 500mA, Package_TO_SOT_SMD:SOT-23-5, symbol Regulator_Linear:AP131-15
- removed U3: RP2040, RP2040_minimal:RP2040-QFN-56, symbol MCU_RaspberryPi_RP2040:RP2040
- removed Y1: 3225_4P 12MHz, Crystal:Crystal_SMD_3225-4Pin_3.2x2.5mm, symbol Device:Crystal_GND24
- added SW1, SW2: SKRK, Button_Switch_SMD:SW_SPST_CK_KXT3, symbol Switch:SW_Push
- added U2: PGA2040, yuiop:PGA2040, symbol yuiop:PGA2040
- C9: value 0.1uf -> 0.1uf 0805
- D_100, D_101, D_102, D_103, D_104, D_105, D_106, D_107, D_108, D_109, D_110, D_111, D_112, D_113, D_114, D_115, D_116, D_117, D_12, D_13, D_14, D_15, D_16, D_17, D_18, D_19, D_20, D_21, D_22, D_23, D_24, D_25, D_26, D_27, D_28, D_29, D_30, D_31, D_32, D_33, D_34, D_35, D_36, D_37, D_38, D_39, D_40, D_41, D_42, D_43, D_44, D_45, D_46, D_47, D_48, D_49, D_50, D_51, D_52, D_53, D_54, D_55, D_56, D_57, D_58, D_59, D_60, D_61, D_62, D_63, D_64, D_65, D_66, D_67, D_68, D_69, D_70, D_71, D_72, D_73, D_74, D_75, D_76, D_77, D_78, D_79, D_80, D_81, D_82, D_83, D_84, D_85, D_86, D_87, D_88, D_89, D_90, D_91, D_92, D_93, D_94, D_95, D_96, D_97, D_98, D_99: value SOD-123 -> 1N4148W
- R5, R6: value 5.1K 0402 -> 5.1K 0805
- R8: value 330r -> 330r 0805
Connections:
- net GND: now also SW1.1, SW2.1, U2.11 (GND), U2.12 (GND), U2.23 (GND), U2.24 (GND), U2.35 (GND), U2.36 (GND), U2.47 (GND), U2.48 (GND)
- net RUN: now also SW1.2, U2.42 (RUN)
- net SWCLK: now also U2.41 (SWCLK)
- net SWD: now also U2.39 (SWDIO)
- net USB_D+: now also U2.40 (USB_DP)
- net USB_D-: now also U2.38 (USB_DM)
- net VBUS: now also U2.46 (VBUS)
- net col0: now also U2.2 (UART1)
- net col1: now also U2.3 (GPIO2)
- net col10: now also U2.14 (GPIO11)
- net col11: now also U2.15 (GPIO12)
- net col12: now also U2.16 (GPIO13)
- net col13: now also U2.17 (GPIO14)
- net col14: now also U2.18 (GPIO15)
- net col15: now also U2.19 (GPIO16)
- net col16: now also U2.20 (GPIO17)
- net col17: now also U2.21 (GPIO18)
- net col19: now also U2.22 (GPIO19)
- net col2: now also U2.4 (GPIO3)
- net col20: now also U2.25 (GPIO20)
- net col21: now also U2.26 (GPIO21)
- net col22: now also U2.27 (GPIO22)
- net col3: now also U2.5 (GPIO4)
- net col4: now also U2.6 (GPIO5)
- net col5: now also U2.7 (GPIO6)
- net col6: now also U2.8 (GPIO7)
- net col7: now also U2.9 (GPIO8)
- net col8: now also U2.10 (GPIO9)
- net col9: now also U2.13 (GPIO10)
- net row1: now also U2.1 (UART0)
- net row3: now also U2.28 (GPIO23)
- net row4: now also U2.29 (GPIO24)
- net row5: now also U2.30 (GPIO25)
- net row6: now also U2.31 (ADC26)
- net row7: now also U2.32 (ADC27)
- new net BOOTSEL: SW2.2, U2.37 (BOOTSEL)
Other:
- note removed: "1K resistor to prevent overdriving of the crystal as per the minimal design example"
- note removed: "500mA hold current 1A trip 6V trip"
- note removed: "Crystal"
- note removed: "D1 NEEDS to be 0omh resistor or 1N4002 diode"
- note removed: "Flash"
- note removed: "GD25Q40CEIGR is NOT Compatible you need GD25W16* needs to be a multiple of 8 atleast for circuitpython. (Ive not confirmed if GD25W16 works I just Have some boards with GD25Q40CEIGR and they dont work)"
- note removed: "Im pretty sure a lot of these W25QXXX Chips are pin compatible Dont quote me on that"
- note removed: "Im unsure if the RP2040 can function with flash larger than 128Mb"
- note removed: "MAKE SURE THIS LINE is ran off of pin43 or close to pin43"
- note removed: "Make sure C10 is close to pin 44 of RP2040"
- note removed: "Make sure C3 is close to pin 45 of RP2040"
- note removed: "Make sure R3 and R4 are close to RP2040"
- note removed: "Make sure the flash chip you have selected supports 3.3V power or adjust the design."
- note removed: "Only fit cBP1 if you have selected an alternate voltage regulator TLV75533PDBVR does not require cBP1."
- note removed: "Pin 9 technically doesnt exist its the main central contact under the chip for heat dicipation"
- note removed: "RP2040 supports 1MHz to 15MHz"
- note removed: "These decoupling capacitors are meant to be put close by each 3.3V pin of the RP2040"
- note removed: "Would assume you could just not connect SD2 and SD3 for non QSPI"
- note removed: "https://datasheets.raspberrypi.com/rp2040/hardware-design-with-rp2040.pdf On page 13 you can learn more details of what flash is supported"
- note removed: "not 22pf but pick to match crystal."
- note removed: "suposedly the rp2040 supports SPI-2 flash but I havent tried it."
- note removed: "this is for factory testing always pull this to ground"
- moved on the sheet: J5

Commit message: swapped buttons to Panasonic side buttons  and wired up debug header
Parts:
- SW1, SW2: value SKRK -> EVQP; footprint Button_Switch_SMD:SW_SPST_CK_KXT3 -> Button_Switch_SMD:Panasonic_EVQPUL_EVQPUC
Changed lines of the file:
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@@
       (effects (font (size 1.27 1.27)))
     )
-    (property "Value" "SKRK" (at 31.75 120.65 0)
+    (property "Value" "EVQP" (at 31.75 120.65 0)
       (effects (font (size 1.27 1.27)))
     )
-    (property "Footprint" "Button_Switch_SMD:SW_SPST_CK_KXT3" (at 31.75 120.65 0)
+    (property "Footprint" "Button_Switch_SMD:Panasonic_EVQPUL_EVQPUC" (at 31.75 120.65 0)
       (effects (font (size 1.27 1.27)) hide)
     )
@@
       (effects (font (size 1.27 1.27)))
     )
-    (property "Value" "SKRK" (at 31.75 133.35 0)
+    (property "Value" "EVQP" (at 31.75 133.35 0)
       (effects (font (size 1.27 1.27)))
     )
-    (property "Footprint" "Button_Switch_SMD:SW_SPST_CK_KXT3" (at 31.75 133.35 0)
+    (property "Footprint" "Button_Switch_SMD:Panasonic_EVQPUL_EVQPUC" (at 31.75 133.35 0)
       (effects (font (size 1.27 1.27)) hide)
     )
